Commit message: Commit for task 2 - Checkpoint 1: Introduction to Gazebo

File: my_rb1_description/urdf/my_rb1_description.xacro (robot description, xacro)
@@ -1,4 +1,5 @@
 <?xml version="1.0" ?>
-<robot name="rb1">
+<robot name="rb1" xmlns:xacro="http://www.ros.org/wiki/xacro">
+    <xacro:include filename="$(find my_rb1_description)/urdf/my_rb1_description.gazebo" />
     <material name="blue">
         <color rgba="0 0 1 1"/>
@@ -13,5 +14,5 @@
         <inertial>
             <mass value="10" />
-            <inertia ixx="0.23125"  ixy="0"  ixz="0.3125" iyy="0.23125" iyz="0" izz="0.3125" />
+            <inertia ixx="0.23125"  ixy="0"  ixz="0" iyy="0.23125" iyz="0" izz="0.3125" />
         </inertial>
         <collision>
@@ -54,5 +55,5 @@
         <parent link="base_link" />
         <child link="right_wheel" />
-        <origin xyz="0.0 0.2 -0.15" rpy="0 0 0" />
+        <origin xyz="0 0.2 -0.15" rpy="0 0 0" />
         <axis xyz="0 1 0" />
     </joint>
@@ -63,4 +64,5 @@
         </inertial>
         <collision>
+            <origin xyz="0 0 0" rpy="1.57 0 0" />
             <geometry>
                 <cylinder radius="0.025" length="0.03" />
@@ -78,5 +80,5 @@
         <parent link="base_link" />
         <child link="left_wheel" />
-        <origin xyz="0.0 -0.2 -0.15" rpy="0 0 0" />
+        <origin xyz="0 -0.2 -0.15" rpy="0 0 0" />
         <axis xyz="0 1 0" />
     </joint>
@@ -87,4 +89,5 @@
         </inertial>
         <collision>
+            <origin xyz="0 0 0" rpy="1.57 0 0" />
             <geometry>
                 <cylinder radius="0.025" length="0.03" />

Commit message: Commit for task 3- Checkpoint: 1 Introduction to Gazebo

File: my_rb1_description/urdf/my_rb1_description.xacro (robot description, xacro)
@@ -13,6 +13,6 @@
     <link name="base_link">
         <inertial>
-            <mass value="10" />
-            <inertia ixx="0.23125"  ixy="0"  ixz="0" iyy="0.23125" iyz="0" izz="0.3125" />
+            <mass value="23" />
+            <inertia ixx="0.531875"  ixy="0"  ixz="0" iyy="0.531875" iyz="0" izz="0.71875" />
         </inertial>
         <collision>
@@ -32,12 +32,13 @@
         <parent link="base_link" />
         <child link="front_laser" />
-        <origin xyz="0.25 0.0 0.075" rpy="0 0 0" />
+        <origin xyz="0.25 0 0.075" rpy="0 0 0" />
     </joint>
     <link name="front_laser">
         <inertial>
-            <mass value="5" />
-            <inertia ixx="0.00115625"  ixy="0"  ixz="0" iyy="0.00115625" iyz="0" izz="0.0015625" />
+            <mass value="0.5" />
+            <inertia ixx="0.000115625"  ixy="0"  ixz="0" iyy="0.000115625" iyz="0" izz="0.00015625" />
         </inertial>
         <collision>
+            <origin xyz="0 0 0" rpy="3.14 0 0" />
             <geometry>
                  <cylinder radius="0.025" length="0.03" />
@@ -55,14 +56,14 @@
         <parent link="base_link" />
         <child link="right_wheel" />
-        <origin xyz="0 0.2 -0.15" rpy="0 0 0" />
+        <origin xyz="0 -0.2 -0.15" rpy="0 0 0" />
         <axis xyz="0 1 0" />
     </joint>
     <link name="right_wheel">
         <inertial>
-            <mass value="2.5" />
-            <inertia ixx="0.000578125"  ixy="0"  ixz="0" iyy="0.000578125" iyz="0" izz="0.00078125" />
+            <mass value="0.5" />
+            <inertia ixx="0.000115625"  ixy="0"  ixz="0" iyy="0.000115625" iyz="0" izz="0.00015625" />
         </inertial>
         <collision>
-            <origin xyz="0 0 0" rpy="1.57 0 0" />
+            <origin xyz="0 0 0" rpy="-1.57 0 0" />
             <geometry>
                 <cylinder radius="0.025" length="0.03" />
@@ -70,5 +71,5 @@
         </collision>
         <visual>
-            <origin xyz="0 0 0" rpy="1.57 0 0" />
+            <origin xyz="0 0 0" rpy="-1.57 0 0" />
             <geometry>
                 <cylinder radius="0.025" length="0.03" />
@@ -80,11 +81,11 @@
         <parent link="base_link" />
         <child link="left_wheel" />
-        <origin xyz="0 -0.2 -0.15" rpy="0 0 0" />
+        <origin xyz="0 0.2 -0.15" rpy="0 0 0" />
         <axis xyz="0 1 0" />
     </joint>
     <link name="left_wheel">
         <inertial>
-            <mass value="2.5" />
-            <inertia ixx="0.000578125"  ixy="0"  ixz="0" iyy="0.000578125" iyz="0" izz="0.00078125" />
+            <mass value="0.5" />
+            <inertia ixx="0.000115625"  ixy="0"  ixz="0" iyy="0.000115625" iyz="0" izz="0.00015625" />
         </inertial>
         <collision>
@@ -105,11 +106,10 @@
         <parent link="base_link" />
         <child link="front_caster" />
-        <origin xyz="0.1 0.0 -0.15" rpy="0 0 0" />
-        <dynamics damping="0.0" friction="0.0" />
+        <origin xyz="0.175 0.0 -0.15" rpy="0 0 0" />
     </joint>
     <link name="front_caster">
         <inertial>
-            <mass value="2.5" />
-            <inertia ixx="0.000625"  ixy="0"  ixz="0" iyy="0.000625" iyz="0" izz="0.000625" />
+            <mass value="0.25" />
+            <inertia ixx="0.0000625" ixy="0" ixz="0" iyy="0.0000625" iyz="0" izz="0.0000625"/>
         </inertial>
         <collision>
@@ -128,11 +128,10 @@
         <parent link="base_link" />
         <child link="back_caster" />
-        <origin xyz="-0.1 0.0 -0.15" rpy="0 0 0" />
-        <dynamics damping="0.0" friction="0.0" />
+        <origin xyz="-0.175 0.0 -0.15" rpy="0 0 0" />
     </joint>
     <link name="back_caster">
         <inertial>
-            <mass value="2.5" />
-            <inertia ixx="0.000625"  ixy="0"  ixz="0" iyy="0.000625" iyz="0" izz="0.000625" />
+            <mass value="0.25" />
+            <inertia ixx="0.0000625" ixy="0" ixz="0" iyy="0.0000625" iyz="0" izz="0.0000625"/>
         </inertial>
         <collision>

Commit message: Task 3 completed

File: my_rb1_description/urdf/my_rb1_description.xacro (robot description, xacro)
@@ -13,6 +13,6 @@
     <link name="base_link">
         <inertial>
-            <mass value="23" />
-            <inertia ixx="0.531875"  ixy="0"  ixz="0" iyy="0.531875" iyz="0" izz="0.71875" />
+            <mass value="20" />
+            <inertia ixx="0.4625"  ixy="0"  ixz="0" iyy="0.4625" iyz="0" izz="0.625" />
         </inertial>
         <collision>
@@ -52,15 +52,40 @@
         </visual>
     </link>
+    <!-- Left Wheel -->
+    <joint name="left_wheel_base_joint" type="continuous">
+        <parent link="base_link" />
+        <child link="left_wheel" />
+        <origin xyz="0 -0.2 -0.15" rpy="0 0 0" />
+        <axis xyz="0 1 0" />
+    </joint>
+    <link name="left_wheel">
+        <inertial>
+            <mass value="2" />
+            <inertia ixx="0.0153125"  ixy="0"  ixz="0" iyy="0.0153125" iyz="0" izz="0.000625" />
+        </inertial>
+        <collision>
+            <origin xyz="0 0 0" rpy="1.57 0 0" />
+            <geometry>
+                <cylinder radius="0.025" length="0.03" />
+            </geometry>
+        </collision>
+        <visual>
+            <origin xyz="0 0 0" rpy="1.57 0 0" />
+            <geometry>
+                <cylinder radius="0.025" length="0.03" />
+            </geometry>
+        </visual>
+    </link>
     <!-- Right Wheel -->
     <joint name="right_wheel_base_joint" type="continuous">
         <parent link="base_link" />
         <child link="right_wheel" />
-        <origin xyz="0 -0.2 -0.15" rpy="0 0 0" />
+        <origin xyz="0 0.2 -0.15" rpy="0 0 0" />
         <axis xyz="0 1 0" />
     </joint>
     <link name="right_wheel">
         <inertial>
-            <mass value="0.5" />
-            <inertia ixx="0.000115625"  ixy="0"  ixz="0" iyy="0.000115625" iyz="0" izz="0.00015625" />
+            <mass value="2" />
+           <inertia ixx="0.0153125"  ixy="0"  ixz="0" iyy="0.0153125" iyz="0" izz="0.000625" />
         </inertial>
         <collision>
@@ -72,29 +97,4 @@
         <visual>
             <origin xyz="0 0 0" rpy="-1.57 0 0" />
-            <geometry>
-                <cylinder radius="0.025" length="0.03" />
-            </geometry>
-        </visual>
-    </link>
-    <!-- Left Wheel -->
-    <joint name="left_wheel_base_joint" type="continuous">
-        <parent link="base_link" />
-        <child link="left_wheel" />
-        <origin xyz="0 0.2 -0.15" rpy="0 0 0" />
-        <axis xyz="0 1 0" />
-    </joint>
-    <link name="left_wheel">
-        <inertial>
-            <mass value="0.5" />
-            <inertia ixx="0.000115625"  ixy="0"  ixz="0" iyy="0.000115625" iyz="0" izz="0.00015625" />
-        </inertial>
-        <collision>
-            <origin xyz="0 0 0" rpy="1.57 0 0" />
-            <geometry>
-                <cylinder radius="0.025" length="0.03" />
-            </geometry>
-        </collision>
-        <visual>
-            <origin xyz="0 0 0" rpy="1.57 0 0" />
             <geometry>
                 <cylinder radius="0.025" length="0.03" />
